Commit message: Fixing the bb gazebo sim

File: src/baebot_sim/urdf/baebot_sim.xacro (robot description, xacro)
@@ -15,15 +15,15 @@
     <pose>0 0 0.1 0 0 0</pose>
     <inertial>
-      <mass value="15"/>
+      <mass value="1"/>
       <origin xyz="0 0 0" rpy="0 0 0"/>
       <inertia
-          ixx="0.08425" ixy="0" ixz="0"
-          iyy="0.318625" iyz="0"
-          izz="0.390625"
+          ixx="0.035" ixy="0" ixz="0"
+          iyy="0.035" iyz="0"
+          izz="0.035"
       />
     </inertial>
     <collision name="chassis_collision">
       <geometry>
-        <box size="0.5 0.25 0.07"/>
+        <box size="0.125 0.125 0.085"/>
       </geometry>
     </collision>
@@ -31,18 +31,18 @@
       <origin rpy="0 0 0" xyz="0 0 0"/>
       <geometry>
-        <box size="0.5 0.25 0.07"/>
+        <box size="0.125 0.125 0.085"/>
       </geometry>
     </visual>
-    <!--front caster-->
+    <!--rear caster-->
     <collision name="front_caster_collision">
-      <origin xyz="0.35 0 -0.05" rpy=" 0 0 0"/>
+      <origin xyz="-0.04 0 -0.035" rpy=" 0 0 0"/>
       <geometry>
-        <sphere radius="0.05"/>
+        <sphere radius="0.015"/>
       </geometry>
     </collision>
     <visual name="front_caster_visual">
-      <origin xyz="0.2 0 -0.05" rpy=" 0 0 0"/>
+      <origin xyz="-0.04 0 -0.035" rpy=" 0 0 0"/>
       <geometry>
-        <sphere radius="0.05"/>
+        <sphere radius="0.015"/>
       </geometry>
     </visual>
@@ -51,16 +51,16 @@
   <link name='left_wheel'>
     <inertial>
-      <mass value="5"/>
+      <mass value="0.1"/>
       <origin xyz="0 0 0" rpy="0 1.5707 1.5707" />
       <inertia
-          ixx="0.01354166666" ixy="0" ixz="0"
-          iyy="0.01354166666" iyz="0"
-          izz="0.025"
+          ixx="0.015" ixy="0" ixz="0"
+          iyy="0.015" iyz="0"
+          izz="0.013"
       />
     </inertial>
     <collision name='left_wheel_collision'>
-      <origin  xyz="0 0 0" rpy="0 1.5707 1.5707"/>
+      <origin xyz="0 0 0" rpy="0 1.5707 1.5707"/>
       <geometry>
-        <cylinder length="0.05" radius="0.1"/>
+        <cylinder length="0.025" radius="0.03"/>
       </geometry>
     </collision>
@@ -68,5 +68,5 @@
       <origin xyz="0 0 0" rpy="0 1.5707 1.5707"/>
       <geometry>
-        <cylinder length="0.05" radius="0.1"/>
+        <cylinder length="0.025" radius="0.03"/>
       </geometry>
     </visual>
@@ -74,9 +74,9 @@
   <!--Joint (left_wheel_hinge)-->
   <joint name="left_wheel_hinge" type="continuous">
-    <origin xyz="-0.05 0.15 0" rpy="0 0 0"/>
+    <origin xyz="0.035 0.078 -0.02" rpy="0 0 0"/>
     <child link="left_wheel" />
     <parent link="chassis"/>
     <axis xyz="0 1 0" rpy="0 0 0" />
-    <limit effort="10000" velocity="1000"/>
+    <limit effort="1" velocity="1.5"/>
     <joint_properties damping="1.0" friction="1.0" />
   </joint>
@@ -85,9 +85,9 @@
     <inertial>
       <origin xyz="0 0 0" rpy="0 1.5707 1.5707" />
-      <mass value="5"/>
+      <mass value="0.1"/>
       <inertia
-          ixx="0.01354166666" ixy="0" ixz="0"
-          iyy="0.01354166666" iyz="0"
-          izz="0.025"
+          ixx="0.015" ixy="0" ixz="0"
+          iyy="0.015" iyz="0"
+          izz="0.013"
       />
     </inertial>
@@ -95,5 +95,5 @@
       <origin xyz="0 0 0" rpy="0 1.5707 1.5707"/>
       <geometry>
-        <cylinder length="0.05" radius="0.1"/>
+        <cylinder length="0.025" radius="0.03"/>
       </geometry>
     </collision>
@@ -101,5 +101,5 @@
       <origin xyz="0 0 0" rpy="0 1.5707 1.5707"/>
       <geometry>
-        <cylinder length="0.05" radius="0.1"/>
+        <cylinder length="0.025" radius="0.03"/>
       </geometry>
     </visual>
@@ -107,9 +107,9 @@
   <!--Joint (right_wheel_hinge)-->
   <joint name="right_wheel_hinge" type="continuous">
-    <origin xyz="-0.05 -0.15 0" rpy="0 0 0"/>
+    <origin xyz="0.035 -0.078 -0.02" rpy="0 0 0"/>
     <child link="right_wheel" />
     <parent link="chassis"/>
     <axis rpy="0 0 0" xyz="0 1 0"/>
-    <limit effort="10000" velocity="1000"/>
+    <limit effort="1" velocity="1.5"/>
     <joint_properties damping="1.0" friction="1.0" />
   </joint>
@@ -118,5 +118,5 @@
     <inertial>
       <origin xyz="0 0 0" rpy="0 0 0"/>
-      <mass value="0.1"/>
+      <mass value="0.05"/>
       <box_inertia m="0.1" x="0.05" y="0.05" z="0.05"/>
       <inertia
@@ -129,5 +129,5 @@
       <origin xyz="0 0 0" rpy="0 0 0"/>
       <geometry>
-        <box size=".05 .05 .05"/>
+        <box size=".001 .025 .025"/>
       </geometry>
     </visual>
@@ -135,5 +135,5 @@
       <origin xyz="0 0 0" rpy="0 0 0"/>
       <geometry>
-        <box size=".05 .05 .05"/>
+        <box size=".001 .025 .025"/>
       </geometry>
     </collision>
@@ -141,5 +141,5 @@
   <!--Joint (camera)-->
   <joint type="fixed" name="camera_joint">
-    <origin xyz="0.25 0 0" rpy="0 0 0"/>
+    <origin xyz="0.063 0 0" rpy="0 0 0"/>
     <child link="camera"/>
     <parent link="chassis"/>
@@ -160,5 +160,5 @@
       <origin xyz="0 0 0" rpy="0 0 0"/>
       <geometry>
-        <mesh filename="package://my_robot/meshes/hokuyo.dae"/>
+        <mesh filename="package://baebot_sim/meshes/hokuyo.dae"/>
       </geometry>
     </visual>
@@ -172,5 +172,5 @@
   <!--Joint (hokuyo)-->
   <joint type="fixed" name="hokuyo_joint">
-    <origin xyz="0.2 0 .07" rpy="0 0 0"/>
+    <origin xyz="0.037 0 .078" rpy="0 0 0"/>
     <child link="hokuyo"/>
     <parent link="chassis"/>
@@ -182,8 +182,8 @@
   </gazebo>
   <gazebo reference="left_wheel">
-    <material>Gazebo/Black</material>
+    <material>Gazebo/White</material>
   </gazebo>
   <gazebo reference="right_wheel">
-    <material>Gazebo/Black</material>
+    <material>Gazebo/White</material>
   </gazebo>
   <gazebo reference="camera">
@@ -191,5 +191,5 @@
   </gazebo>
   <gazebo reference="hokuyo">
-    <material>Gazebo/Black</material>
+    <material>Gazebo/Yellow</material>
   </gazebo>
 </robot>

Commit message: fine tuning baebot sim

File: src/baebot_sim/urdf/baebot_sim.xacro (robot description, xacro)
@@ -13,17 +13,17 @@
   <!--Link (chasiss)-->
   <link name="chassis">
-    <pose>0 0 0.1 0 0 0</pose>
+    <pose>0 0 0.05 0 0 0</pose>
     <inertial>
-      <mass value="1"/>
+      <mass value="0.8"/>
       <origin xyz="0 0 0" rpy="0 0 0"/>
       <inertia
-          ixx="0.035" ixy="0" ixz="0"
-          iyy="0.035" iyz="0"
-          izz="0.035"
+          ixx="0.152" ixy="0" ixz="0"
+          iyy="0.144" iyz="0"
+          izz="0.2"
       />
     </inertial>
     <collision name="chassis_collision">
       <geometry>
-        <box size="0.125 0.125 0.085"/>
+        <box size="0.12 0.125 0.085"/>
       </geometry>
     </collision>
@@ -31,18 +31,18 @@
       <origin rpy="0 0 0" xyz="0 0 0"/>
       <geometry>
-        <box size="0.125 0.125 0.085"/>
+        <box size="0.12 0.125 0.085"/>
       </geometry>
     </visual>
     <!--rear caster-->
     <collision name="front_caster_collision">
-      <origin xyz="-0.04 0 -0.035" rpy=" 0 0 0"/>
+      <origin xyz="-0.0475 0 -0.04" rpy=" 0 0 0"/>
       <geometry>
-        <sphere radius="0.015"/>
+        <sphere radius="0.01"/>
       </geometry>
     </collision>
     <visual name="front_caster_visual">
-      <origin xyz="-0.04 0 -0.035" rpy=" 0 0 0"/>
+      <origin xyz="-0.0475 0 -0.04" rpy=" 0 0 0"/>
       <geometry>
-        <sphere radius="0.015"/>
+        <sphere radius="0.01"/>
       </geometry>
     </visual>
@@ -51,10 +51,10 @@
   <link name='left_wheel'>
     <inertial>
-      <mass value="0.1"/>
+      <mass value="0.05"/>
       <origin xyz="0 0 0" rpy="0 1.5707 1.5707" />
       <inertia
           ixx="0.015" ixy="0" ixz="0"
           iyy="0.015" iyz="0"
-          izz="0.013"
+          izz="0.0044"
       />
     </inertial>
@@ -62,5 +62,5 @@
       <origin xyz="0 0 0" rpy="0 1.5707 1.5707"/>
       <geometry>
-        <cylinder length="0.025" radius="0.03"/>
+        <cylinder length="0.025" radius="0.0325"/>
       </geometry>
     </collision>
@@ -68,5 +68,5 @@
       <origin xyz="0 0 0" rpy="0 1.5707 1.5707"/>
       <geometry>
-        <cylinder length="0.025" radius="0.03"/>
+        <cylinder length="0.025" radius="0.0325"/>
       </geometry>
     </visual>
@@ -79,5 +79,5 @@
     <axis xyz="0 1 0" rpy="0 0 0" />
     <limit effort="1" velocity="1.5"/>
-    <joint_properties damping="1.0" friction="1.0" />
+    <joint_properties damping="0" friction="0" />
   </joint>
   <!--Link (right_wheel)-->
@@ -85,9 +85,9 @@
     <inertial>
       <origin xyz="0 0 0" rpy="0 1.5707 1.5707" />
-      <mass value="0.1"/>
+      <mass value="0.05"/>
       <inertia
           ixx="0.015" ixy="0" ixz="0"
           iyy="0.015" iyz="0"
-          izz="0.013"
+          izz="0.0044"
       />
     </inertial>
@@ -95,5 +95,5 @@
       <origin xyz="0 0 0" rpy="0 1.5707 1.5707"/>
       <geometry>
-        <cylinder length="0.025" radius="0.03"/>
+        <cylinder length="0.025" radius="0.0325"/>
       </geometry>
     </collision>
@@ -101,5 +101,5 @@
       <origin xyz="0 0 0" rpy="0 1.5707 1.5707"/>
       <geometry>
-        <cylinder length="0.025" radius="0.03"/>
+        <cylinder length="0.025" radius="0.0325"/>
       </geometry>
     </visual>
@@ -112,5 +112,5 @@
     <axis rpy="0 0 0" xyz="0 1 0"/>
     <limit effort="1" velocity="1.5"/>
-    <joint_properties damping="1.0" friction="1.0" />
+    <joint_properties damping="0" friction="0" />
   </joint>
   <!--Link (camera)-->
@@ -118,10 +118,10 @@
     <inertial>
       <origin xyz="0 0 0" rpy="0 0 0"/>
-      <mass value="0.05"/>
-      <box_inertia m="0.1" x="0.05" y="0.05" z="0.05"/>
+      <mass value="0.001"/>
+      <!--box_inertia m="0.001" x="0.001" y="0.025" z="0.025"/-->
       <inertia
-          ixx="1e-6" ixy="0" ixz="0"
-          iyy="1e-6" iyz="0"
-          izz="1e-6"
+          ixx="1e-9" ixy="0" ixz="0"
+          iyy="1e-9" iyz="0"
+          izz="1e-9"
       />
     </inertial>
@@ -141,5 +141,5 @@
   <!--Joint (camera)-->
   <joint type="fixed" name="camera_joint">
-    <origin xyz="0.063 0 0" rpy="0 0 0"/>
+    <origin xyz="0.061 0 0" rpy="0 0 0"/>
     <child link="camera"/>
     <parent link="chassis"/>
@@ -150,5 +150,5 @@
     <inertial>
       <origin xyz="0 0 0" rpy="0 0 0"/>
-      <mass value="1e-5"/>
+      <mass value="0.1"/>
       <inertia
           ixx="1e-6" ixy="0" ixz="0"
@@ -172,5 +172,5 @@
   <!--Joint (hokuyo)-->
   <joint type="fixed" name="hokuyo_joint">
-    <origin xyz="0.037 0 .078" rpy="0 0 0"/>
+    <origin xyz="0.03 0 .078" rpy="0 0 0"/>
     <child link="hokuyo"/>
     <parent link="chassis"/>
